File: BMS/BMS.kicad_sch (KiCad schematic)
At the start: 91 parts, among them IC1 L9963E-TR

Commit message: Schematic updated 3.1.25
Parts:
- removed BT1, BT10, BT11, BT12, BT13, BT14, BT2, BT3, BT4, BT5, BT6, BT7, BT8, BT9: Battery_Cell, symbol Device:Battery_Cell
- removed CESD1, CESD14: 47nf, symbol Device:C_Small
- removed RSense: 100u, symbol Device:R_US
- added CESD17, CESD18, CESD19: 47nf, symbol Device:C_Small
- added CFLTH, CVTREF: C_Small, symbol Device:C_Small
- added CNTC, CNTC1, CNTC2, CNTC3, CNTC4, CNTC5, CNTC6: ~, symbol Device:C_Small
- added DOPT, DZBAT: D_Zener, symbol Device:D_Zener
- added RBAT_DOWN, RFAULTL, RFAULT_DOWN, RFLT, RFLT_PD, RVTREF, RVTREF1, RVTREF2, RVTREF3, RVTREF4, RVTREF5, RVTREF6: R_US, symbol Device:R_US
- added RGPIO, RGPIO1, RGPIO2, RGPIO3, RGPIO4, RGPIO5, RGPIO6, RTERM, RTERM1: ~, symbol Device:R_US
- added T1, T2: Transformer_1P_1S, symbol Device:Transformer_1P_1S
- added U1: QRE1113GR, OptoDevice:Everlight_ITR1201SR10AR, symbol Sensor_Proximity:QRE1113GR
Connections:
- net AGND: now also CESD13.1, U1.2 (K)
- net GNDESD: now also CESD17.2, CESD18.2, CESD19.2, CFLTH.2, DZBAT.2 (A)
- net at IC1.44 (B8_7), RLPF11.2: now also CESD4.1; no longer CESD7.1
- net at RDIS6.2, RDIS7.2, RLPF6.2: now also CESD3.1; no longer CESD6.1
- net at RDIS2.2, RDIS3.2, RLPF3.2: now also CESD18.1; no longer CESD3.1
- net at IC1.29 (B2_1), RLPF2.2: now also CESD19.1; no longer CESD2.1
- net at 4.7uf.1, IC1.18 (VREG), MREG.3 (S): no longer IC1.17 (NPNDRV), IC1.19 (VTREF), MREG.2 (G)
- net at IC1.49 (B10_9), RLPF12.2: now also CESD6.1; no longer CESD9.1
- net at RDIS10.2, RDIS11.2, RLPF8.2: now also CESD8.1; no longer CESD10.1
- net at RDIS8.2, RDIS9.2, RLPF7.2: now also CESD7.1; no longer CESD8.1
- net at IC1.34 (B4_3), RLPF4.2: now also CESD2.1; no longer CESD4.1
- net at RDIS12.2, RDIS13.2, RLPF9.2: now also CESD10.1; no longer CESD12.1
- net at IC1.59 (B14_13), RLPF14.2: now also CESD11.1; no longer CESD13.1
- net at RDIS4.2, RDIS5.2, RLPF5.2: now also CESD17.1
- net at IC1.54 (B12_11), RLPF13.2: now also CESD9.1; no longer CESD11.1
- net at FR_BAT.2, RBAT_UP.1, RDIS14.2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: now also CESD12.1
- net at IC1.1 (GPIO8__SCK): now also CNTC5.2, RGPIO5.2
- net at IC1.10 (GPIO1__FAULTH): now also CFLTH.1, DZBAT.1 (K), RFLT.2, RFLT_PD.2
- net at IC1.11 (GPIO2__FAULTL): now also RFAULTL.2
- net at IC1.12 (GPIO3): now also CNTC.2, RGPIO.2
- net at IC1.13 (GPIO4): now also CNTC1.2, RGPIO1.2
- net at IC1.14 (GPIO5): now also CNTC2.2, RGPIO2.2
- net at IC1.15 (GPIO6): now also CNTC3.2, RGPIO3.2
- net at IC1.16 (GPIO7__WAKEUP): now also CNTC4.2, RGPIO4.2
- net at IC1.2 (GPIO9__SDO): now also CNTC6.2, RGPIO6.2
- net at IC1.3 (ISOLP_SDI): now also RTERM.2, T1.2 (AB)
- net at IC1.4 (ISOLM_NCS): now also RTERM.1, T1.1 (AA)
- net at IC1.7 (ISOHP): now also RTERM1.2, T2.2 (AB)
- net at IC1.8 (ISOHM): now also RTERM1.1, T2.1 (AA)
- new net: RGPIO3.1, RVTREF3.1
- new net: DOPT.2 (A), RFAULT_DOWN.1, U1.4
- new net: CVTREF.1, IC1.19 (VTREF), RVTREF.2, RVTREF1.2, RVTREF2.2, RVTREF3.2, RVTREF4.2, RVTREF5.1, RVTREF6.1
- new net: RGPIO5.1, RVTREF6.2
- new net: RGPIO.1, RVTREF.1
- new net: RGPIO1.1, RVTREF1.1
- new net: RGPIO6.1, RVTREF5.2
- new net: RGPIO2.1, RVTREF2.1
- new net: DOPT.1 (K), RBAT_DOWN.2, U1.3
- new net: RGPIO4.1, RVTREF4.1
- new net: IC1.17 (NPNDRV), MREG.2 (G)
- new net: RFAULTL.1, U1.1 (A)
- new net GNDREF: CNTC.1, CNTC1.1, CNTC2.1, CNTC3.1, CNTC4.1, CNTC5.1, CNTC6.1, CVTREF.2, RFLT_PD.1
Other:
- note added: "We Need to get a model for the actual Optocoupler (PS2703-1-F3-K-A is recommendend in the data sheet)"
- note removed: "Battery+"
- note removed: "GPIO connection"
- moved on the sheet: CBOOT, CESD5
