File: RF System/Magnetometer Dev Board/Magnetometer Dev Board.kicad_pcb (KiCad board)
At the start: 2 copper layers, 22 x 27.5 mm, 5 parts, among them J1 Conn_01x10_Pin, U1 BMM350

Commit message: RF + Telem (#9)
Co-authored-by: weijing-c <128620043+weijing-c@users.noreply.github.com>
Parts:
- C1, C2: footprint Capacitor_SMD:C_0603_1608Metric -> Capacitor_SMD:C_0805_2012Metric
- C3: footprint Capacitor_SMD:C_0402_1005Metric -> Capacitor_SMD:C_0805_2012Metric
- moved C1 0.50 mm to (118.0, 85.5)
- moved C3 0.50 mm to (118.5, 92.0)
Other:
- board size 22 x 27.5 mm -> 22 x 28 mm
