File: megaTC_dev_board/megaTC_dev_board/megaTC_dev_board.kicad_pcb (KiCad board)
At the start: 2 copper layers, 19 parts, among them J1 Conn_01x08_Pin, J2 Conn_01x08_Pin, J3 Conn_01x08_Pin, U1 LTC2984CLX-PBF, U2 TPD4E1B06DCKR, U3 TPD4E1B06DCKR, U4 TPD4E1B06DCKR, U5 TPD4E1B06DCKR, U6 TPD4E1B06DCKR

Commit message: routing routingghsdjadsd
Parts:
- added C10: 0.01uF, Capacitor_SMD:C_0603_1608Metric, B.Cu at (158.4, 106.0)
- added C11: 0.01uF, Capacitor_SMD:C_0603_1608Metric, B.Cu at (158.4, 103.2)
- added C12: 0.01uF, Capacitor_SMD:C_0603_1608Metric, B.Cu at (158.4, 100.5)
- added C13: 0.01uF, Capacitor_SMD:C_0603_1608Metric, F.Cu at (181.5, 100.0)
- added C14: 0.01uF, Capacitor_SMD:C_0603_1608Metric, F.Cu at (181.5, 102.5)
- added C15: 0.01uF, Capacitor_SMD:C_0603_1608Metric, F.Cu at (181.5, 105.0)
- added C16: 0.01uF, Capacitor_SMD:C_0603_1608Metric, F.Cu at (181.5, 107.5)
- added C17: 0.01uF, Capacitor_SMD:C_0603_1608Metric, F.Cu at (181.5, 110.0)
- added C18: 0.01uF, Capacitor_SMD:C_0603_1608Metric, F.Cu at (185.5, 100.0)
- added C19: 0.01uF, Capacitor_SMD:C_0603_1608Metric, F.Cu at (185.5, 102.5)
- added C20: 0.01uF, Capacitor_SMD:C_0603_1608Metric, F.Cu at (185.5, 105.0)
- added C21: 0.01uF, Capacitor_SMD:C_0603_1608Metric, F.Cu at (185.5, 107.5)
- added C8: 0.01uF, Capacitor_SMD:C_0603_1608Metric, B.Cu at (158.4, 111.5)
- added C9: 0.01uF, Capacitor_SMD:C_0603_1608Metric, B.Cu at (158.5, 108.8)
- added R3: 10k, Resistor_SMD:R_0603_1608Metric, F.Cu at (153.7, 110.0)
- added R4: 10k, Resistor_SMD:R_0603_1608Metric, F.Cu at (153.7, 112.5)
Connections:
- J1 pad 8: CH8 -> COMMON
- J2 pad 2: CH9 -> CH10
- J2 pad 3: CH10 -> CH11
- J2 pad 4: CH11 -> CH12
- J2 pad 5: CH12 -> CH13
- J2 pad 6: CH13 -> CH14
- J2 pad 7: CH14 -> CH15
- J2 pad 8: CH15 -> COMMON
- U3 pad 5: CH9 -> CH10
- U4 pad 1: CH10 -> CH11
- U4 pad 2: CH11 -> CH12
- U4 pad 4: CH12 -> CH13
- U4 pad 5: CH13 -> CH14
- U5 pad 1: CH14 -> CH15
- U5 pad 2: CH15 -> RESET_LOW
- U5 pad 4: RESET_LOW -> CS_LOW
- U5 pad 5: CS_LOW -> SDI
- U6 pad 1: SDI -> SDO
- U6 pad 2: SDO -> SCK
- U6 pad 4: SCK -> INTERRUPT
- U6 pad 5: INTERRUPT -> COMMON
Routing:
- net CH9: track 10.9 -> 0.00 mm
- net CH14: track 10.6 -> 6.03 mm
- net CH10: track 6.57 -> 10.9 mm
- net COMMON: track 0.00 -> 3.49 mm
- net SCK: track 3.86 -> 6.94 mm
- net CH15: track 7.77 -> 10.6 mm
- net RESET_LOW: track 4.68 -> 6.21 mm
- net CH12: track 5.17 -> 6.05 mm
- net CH13: track 6.03 -> 5.17 mm
- net SDO: track 6.36 -> 6.96 mm
- net CH11: track 6.05 -> 6.57 mm

Commit message: push so i can work on my pc lmao
Parts:
- C13, C14, C18: moved to B.Cu
- moved C18 33.3 mm to (153.0, 107.5), turned to -90 degrees
- moved C14 31.6 mm to (150.2, 107.5), turned to -90 degrees
- moved C15 30.3 mm to (151.2, 107.5), turned to -90 degrees
- moved R1 24.5 mm to (149.3, 90.0), turned to 0 degrees
- moved C13 21.2 mm to (160.3, 99.2)
- moved C1 9.92 mm to (141.5, 100.2), turned to 90 degrees
- moved R4 9.55 mm to (144.2, 113.5)
- moved C11 8.71 mm to (164.2, 109.7), turned to -90 degrees
- moved C12 7.99 mm to (164.2, 106.0), turned to -90 degrees
- moved C8 5.53 mm to (158.8, 106.0), turned to -90 degrees
- moved R3 5.28 mm to (149.2, 112.8)
- moved C3 4.26 mm to (146.0, 107.5), turned to -90 degrees
- moved C2 4.24 mm to (137.5, 101.2)
- moved C9 3.18 mm to (161.5, 109.7), turned to -90 degrees
- moved C10 3.08 mm to (161.5, 106.0), turned to -90 degrees
Routing:
- net CH15: track 10.6 -> 49.5 mm, vias 0 -> 1
- net CH13: track 5.17 -> 33.9 mm, vias 0 -> 1
- net CH14: track 6.03 -> 33.5 mm, vias 0 -> 1
- net CH12: track 6.05 -> 32.9 mm, vias 0 -> 1
- net CH10: track 10.9 -> 35.2 mm, vias 0 -> 1
- net CH11: track 6.57 -> 30.8 mm, vias 0 -> 1
- net Net-(U1-VREFOUT): track 0.00 -> 4.72 mm
- net +5V: track 0.00 -> 4.64 mm
- net GND: track 0.00 -> 4.36 mm
- net CH3: track 6.37 -> 9.83 mm
- net CH2: track 6.55 -> 9.81 mm, vias 0 -> 1
- added copper zone on In2.Cu, net +5V
- added copper zone on In1.Cu, net GND
Other:
- copper layers 2 -> 4

Commit message: routing routing routignrdhroitu
Parts:
- C15, C16, C17, C19, C20, C21, C4, C5, D1: moved to B.Cu
- moved C16 42.9 mm to (139.0, 113.8), turned to 180 degrees
- moved C17 37.4 mm to (144.3, 113.8), turned to 180 degrees
- moved C19 33.1 mm to (153.2, 110.0), turned to -90 degrees
- moved C20 29.9 mm to (156.0, 110.0), turned to -90 degrees
- moved C21 29.5 mm to (156.0, 106.0), turned to -90 degrees
- moved R2 22.5 mm to (193.2, 95.0), turned to 180 degrees
- moved D2 22.3 mm to (189.1, 95.0)
- moved R3 20.6 mm to (130.2, 104.8)
- moved C15 12.7 mm to (139.0, 111.0), turned to 180 degrees
- moved R4 11.4 mm to (134.4, 107.5)
- moved C14 6.98 mm to (144.2, 111.0), turned to 180 degrees
- moved C5 6.79 mm to (146.0, 92.2), turned to 180 degrees
- moved C4 6.56 mm to (149.8, 92.2), turned to 0 degrees
- moved D1 4.11 mm to (144.5, 106.8), turned to 0 degrees
- moved C18 3.54 mm to (150.5, 110.0)
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Routing:
- net INTERRUPT: track 5.57 -> 47.3 mm
- net CH4: track 5.88 -> 35.6 mm, vias 0 -> 1
- net GND: track 4.36 -> 33.4 mm, vias 0 -> 20
- net CH5: track 5.84 -> 34.0 mm, vias 0 -> 1
- net CH3: track 9.83 -> 35.2 mm, vias 0 -> 1
- net CH8: track 5.57 -> 30.5 mm, vias 0 -> 1
- net CH2: track 9.81 -> 33.8 mm
- net CH7: track 7.02 -> 29.3 mm, vias 0 -> 1
- net SDI: track 6.49 -> 27.5 mm
- net CH6: track 7.33 -> 28.3 mm, vias 0 -> 1
- net SDO: track 6.96 -> 26.9 mm
- net SCK: track 6.94 -> 25.8 mm
- net +5V: track 4.64 -> 14.6 mm, vias 0 -> 6
- net CH9: track 0.00 -> 5.41 mm, vias 0 -> 1
- net COMMON: track 3.49 -> 7.95 mm, vias 0 -> 1
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
Commit message: routing wrap
Parts:
- C4: moved to F.Cu
- C6, R1, R3, R4: moved to B.Cu
- moved R3 20.5 mm to (150.5, 101.8), turned to -90 degrees
- moved R4 19.7 mm to (153.2, 101.8), turned to -90 degrees
- moved C6 16.9 mm to (152.3, 98.2)
- moved R1 11.4 mm to (160.4, 95.0)
- moved C1 6.51 mm to (141.8, 93.8), turned to 0 degrees
- moved C5 6.41 mm to (148.3, 98.2), turned to 0 degrees
- moved D2 4.26 mm to (184.8, 95.2)
- moved R2 4.26 mm to (188.9, 95.2)
- moved C2 2.83 mm to (139.5, 103.2), turned to 90 degrees
- moved C4 1.72 mm to (148.2, 91.5), turned to 180 degrees
Connections:
- U3 pad 4: CH8 -> COMMON
Routing:
- net COMMON: track 7.95 -> 127.4 mm, vias 1 -> 3
- net RESET_LOW: track 6.21 -> 72.6 mm, vias 0 -> 2
- net CS_LOW: track 5.46 -> 67.1 mm, vias 0 -> 2
- net GND: track 33.4 -> 93.9 mm
- net SDI: track 27.5 -> 66.4 mm, vias 0 -> 2
- net SDO: track 26.9 -> 61.9 mm, vias 0 -> 2
- net SCK: track 25.8 -> 59.5 mm, vias 0 -> 2
- net +5V: track 14.6 -> 30.7 mm, vias 6 -> 8
- net Net-(U1-Q3): track 0.00 -> 12.5 mm, vias 0 -> 1
- net CH8: track 30.5 -> 18.8 mm
- net Net-(U1-Q2): track 0.00 -> 9.78 mm, vias 0 -> 1
- net INTERRUPT: track 47.3 -> 56.4 mm
- net Net-(U1-Q1): track 0.00 -> 8.24 mm, vias 0 -> 1
- net Net-(U1-VREF_BYP): track 0.00 -> 6.33 mm
- net CH9: track 5.41 -> 11.5 mm
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Other:
- board outline added: 72.8 x 36.5 mm
- board text added: "Moses Dilts 2025 DAQ TC-RTD Dev"

Commit message: sync
Parts:
- D1: moved to F.Cu
- moved D1 3.62 mm to (148.0, 107.5), turned to 90 degrees
- moved C2 2.55 mm to (142.0, 102.7)
- moved C1 1.03 mm to (142.5, 94.5)
Routing:
- net GND: track 93.9 -> 84.1 mm, vias 20 -> 21
- net +5V: track 30.7 -> 25.7 mm
- net Net-(U1-Q3): track 12.5 -> 8.72 mm
- net CH1: track 5.81 -> 3.06 mm, vias 1 -> 0
- net Net-(U1-VREF_BYP): track 6.33 -> 3.67 mm
- net Net-(U1-Q2): track 9.78 -> 7.65 mm
- net Net-(U1-Q1): track 8.24 -> 6.83 mm
- added copper zone on B.Cu, net GND
- added copper zone on F.Cu, net GND
- added copper zone on In2.Cu, net GND

Commit message: routing updates
Parts:
- C10, C11, C12, C13, C14, C15, C16, C17, C18, C19, C5, C6, C8, C9, R1: moved to F.Cu
- U2, U3, U4, U5, U6: moved to B.Cu
- moved R2 50.0 mm to (142.8, 114.5), turned to 0 degrees
- moved D2 45.5 mm to (142.8, 112.8)
- moved J3 41.3 mm to (143.0, 98.2)
- moved U5 33.7 mm to (147.8, 102.0)
- moved U6 29.3 mm to (160.1, 102.6)
- moved R1 18.7 mm to (142.8, 101.2)
- moved C8 17.0 mm to (163.8, 122.2)
- moved C10 16.3 mm to (160.2, 122.2)
- moved J1 15.4 mm to (143.0, 128.0)
- moved C1 15.0 mm to (155.7, 101.5)
- moved J2 14.5 mm to (166.8, 122.0), turned to 180 degrees
- moved C14 14.1 mm to (142.8, 125.0)
- moved C17 13.8 mm to (152.2, 125.0)
- moved C2 13.5 mm to (142.8, 116.2), turned to 0 degrees
- moved C13 13.5 mm to (160.2, 112.7), turned to -90 degrees
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Routing:
- net COMMON: track 127.4 -> 0.00 mm, vias 3 -> 0
- net RESET_LOW: track 72.6 -> 0.00 mm, vias 2 -> 0
- net CS_LOW: track 67.1 -> 0.00 mm, vias 2 -> 0
- net SDI: track 66.4 -> 0.00 mm, vias 2 -> 0
- net SDO: track 61.9 -> 0.00 mm, vias 2 -> 0
- net SCK: track 59.5 -> 0.00 mm, vias 2 -> 0
- net INTERRUPT: track 56.4 -> 0.00 mm
- net CH15: track 49.5 -> 0.00 mm, vias 1 -> 0
- net GND: track 84.1 -> 37.6 mm
- net CH4: track 35.6 -> 0.00 mm, vias 1 -> 0
- net CH10: track 35.2 -> 0.00 mm, vias 1 -> 0
- net CH13: track 34.1 -> 0.00 mm, vias 1 -> 0
- net CH14: track 33.5 -> 0.00 mm, vias 1 -> 0
- net CH12: track 32.9 -> 0.00 mm, vias 1 -> 0
- net CH11: track 31.1 -> 0.00 mm, vias 1 -> 0
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- removed copper zone on B.Cu, net GND
- removed copper zone on F.Cu, net GND
- removed copper zone on In2.Cu, net GND
Other:
- board outline removed
- board text removed: "Moses Dilts 2025 DAQ TC-RTD Dev"

Commit message: routing progress
Parts:
- C6: moved to B.Cu
- moved C1 16.1 mm to (142.8, 111.0)
- moved C6 7.93 mm to (151.0, 111.2), turned to 0 degrees
- moved C21 7.12 mm to (157.3, 114.5), turned to 0 degrees
- moved U6 6.26 mm to (153.9, 102.2)
- moved C20 4.79 mm to (151.0, 114.5), turned to 180 degrees
- moved U4 4.61 mm to (162.1, 112.9), turned to 90 degrees
- moved C4 4.61 mm to (148.2, 104.5)
- moved R3 3.11 mm to (154.2, 114.5)
- moved R4 3.11 mm to (154.2, 112.8)
- moved U2 2.00 mm to (147.5, 124.2)
- moved U3 1.89 mm to (157.2, 124.2), turned to 0 degrees
- moved C5 1.25 mm to (148.2, 106.8)
- moved U5 0.27 mm to (147.9, 102.2)
- moved R1 0.15 mm to (142.7, 101.2)
Connections:
- U3 pad 5: CH10 -> CH12
- U4 pad 2: CH12 -> CH10
Routing:
- net CH12: track 0.00 -> 25.9 mm, vias 0 -> 1
- net GND: track 37.6 -> 61.6 mm, vias 21 -> 32
- net CH11: track 0.00 -> 21.2 mm, vias 0 -> 2
- net CH13: track 0.00 -> 20.3 mm, vias 0 -> 1
- net CH10: track 0.00 -> 18.7 mm, vias 0 -> 3
- net RESET_LOW: track 0.00 -> 17.4 mm
- net CH14: track 0.00 -> 15.0 mm, vias 0 -> 1
- net SDO: track 0.00 -> 14.8 mm, vias 0 -> 1
- net SCK: track 0.00 -> 13.6 mm, vias 0 -> 1
- net CS_LOW: track 0.00 -> 13.6 mm
- net INTERRUPT: track 0.00 -> 13.5 mm, vias 0 -> 1
- net CH4: track 0.00 -> 13.3 mm, vias 0 -> 1
- net CH15: track 0.00 -> 13.2 mm
- net SDI: track 0.00 -> 12.7 mm
- net CH3: track 6.73 -> 19.3 mm, vias 0 -> 2
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- added copper zone on F.Cu, net GND
Other:
- board text added: "Copperhead TC-RTD Dev 1 Moses Dilts 2025"
- board text added: "RTD in"
- board text added: "SPI in/out"
- board text added: "TC in"

Commit message: routing that is less spahghetti-like wait is that how you spell spahghetti idk i hope so because im committing it rn so it better be right
Parts:
- C4, D1: moved to B.Cu
- U2, U3: moved to F.Cu
- moved C16 9.00 mm to (151.8, 120.8), turned to -90 degrees
- moved D2 8.45 mm to (145.5, 120.8), turned to -90 degrees
- moved D1 8.00 mm to (150.3, 117.0)
- moved C15 7.64 mm to (150.0, 120.8), turned to -90 degrees
- moved C14 6.92 mm to (148.2, 120.8), turned to -90 degrees
- moved R2 6.29 mm to (143.5, 120.8), turned to 90 degrees
- moved C4 5.08 mm to (151.0, 108.8)
- moved C19 4.83 mm to (157.0, 120.8), turned to -90 degrees
- moved C17 4.41 mm to (153.5, 120.8), turned to -90 degrees
- moved C18 3.91 mm to (155.2, 120.8), turned to -90 degrees
- moved C1 2.27 mm to (144.5, 112.5), turned to 180 degrees
- moved U2 2.15 mm to (149.6, 124.6)
- moved C2 1.97 mm to (144.5, 115.2)
- moved C3 1.97 mm to (144.5, 117.0)
- moved U3 0.95 mm to (156.4, 124.6)
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Connections:
- J1 pad 8: COMMON -> GND
- J2 pad 1: COMMON -> GND
- J2 pad 8: COMMON -> GND
Routing:
- net GND: track 61.6 -> 40.0 mm, vias 32 -> 25
- net RESET_LOW: track 17.4 -> 0.53 mm
- net CH10: track 18.7 -> 3.81 mm, vias 3 -> 1
- net CS_LOW: track 13.6 -> 3.33 mm
- net SDI: track 12.7 -> 3.57 mm
- net +5V: track 19.6 -> 12.0 mm, vias 9 -> 8
- net CH12: track 25.9 -> 18.5 mm, vias 1 -> 0
- net CH1: track 9.09 -> 2.81 mm, vias 0 -> 1
- net CH11: track 21.2 -> 15.8 mm, vias 2 -> 1
- net CH3: track 19.3 -> 15.1 mm
- net Net-(U1-LDO): track 6.19 -> 2.58 mm, vias 0 -> 1
- net CH5: track 17.6 -> 14.4 mm
- net COMMON: track 0.00 -> 2.52 mm
- net Net-(U1-VREF_BYP): track 4.69 -> 2.57 mm
- net Net-(U1-VREFOUT): track 6.54 -> 4.57 mm
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