File: flight_computer_b1/flight_computer.kicad_sch (KiCad schematic)
At the start: 11 parts, among them J1 DB25_Socket, J2 DB25_Socket, J3 Conn_01x03, J4 Screw_Terminal_01x02, J5 Pi Connector, J6 Conn_02x02_Odd_Even

Commit message: IC Import
Other:
- added sheet Power Systems (untitled.kicad_sch)
Changed lines of the file:
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@@
+		)
+	)
+	(sheet
+		(at 191.262 61.976)
+		(size 39.624 18.288)
+		(exclude_from_sim no)
+		(in_bom yes)
+		(on_board yes)
+		(dnp no)
+		(fields_autoplaced yes)
+		(stroke
+			(width 0.1524)
+			(type solid)
+		)
+		(fill
+			(color 0 0 0 0.0000)
+		)
+		(property "Sheetname" "Power Systems"
+			(at 191.262 61.2644 0)
+			(effects
+				(font
+					(size 1.27 1.27)
+				)
+				(justify left bottom)
+			)
+		)
+		(property "Sheetfile" "untitled.kicad_sch"
+			(at 191.262 80.8486 0)
+			(effects
+				(font
+					(size 1.27 1.27)
+				)
+				(justify left top)
+				(hide yes)
+			)
+		)
+		(instances
+			(project "flight_computer"
+				(path "/b71a7b79-cdb5-4e38-a72c-0daaa3474f05"
+					(page "20")
+				)
+			)
 		)
 	)
