File: flight_computer_b1/temperature.kicad_sch (KiCad schematic)
At the start: 1 part, among them U10 LTC2983

Commit message: block 1 fc tc updates
Parts:
- added C1, C2, C3, C4: 0.1uF, symbol Device:C
- added C12, C13, C14, C15: 10uF, symbol Device:C
Connections:
- net GND: now also U10.13 (V_{REFOUT}), U10.14 (V_{REFP}), U10.17 (CH2), U10.19 (CH4), U10.21 (CH6), U10.23 (CH8), C1.2, C13.2, C14.2, C15.2, C2.2, C3.2, C4.2
- net VDD: now also U10.42 (~{RESET})
- net at U10.11 (V_{REF_BYP}): now also C14.1
- net TC1+: now reaches U10.16 (CH1)
- net TC1+: now also C1.1
- net TC2+: now reaches U10.18 (CH3)
- net TC2+: now also C2.1
- net TC3+: now reaches U10.20 (CH5)
- net TC3+: now also C3.1
- net TC4+: now reaches U10.22 (CH7)
- net TC4+: now also C4.1
- net RTD1A: now reaches U10.24 (CH9)
- net RTD1B: now reaches U10.25 (CH10)
- net RTD1C: now reaches U10.26 (CH11)
- net RTD2A: now reaches U10.27 (CH12)
- net RTD2B: now reaches U10.28 (CH13)
- net RTD2C: now reaches U10.29 (CH14)
- net INTERRUPT: now reaches U10.37 (INTERRUPT)
- net at U10.43 (LDO): now also C15.1
- net at U10.46 (Q3): now also C13.1
- net at U10.47 (Q2): now also C12.2
- net at U10.48 (Q1): now also C12.1
- no-connect marks 0 -> 6
Other:
- note added: "TC decoupling caps"

Commit message: tc updates
Parts:
- renumbered C1 to C16, C2 to C17, C3 to C18, C4 to C19
Changed lines of the file:
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@@
 		(dnp no)
 		(fields_autoplaced yes)
-		(property "Reference" "C?"
+		(property "Reference" "C17"
 			(at 66.04 78.7399 0)
 			(effects
@@
 			(project "flight_computer"
 				(path "/b71a7b79-cdb5-4e38-a72c-0daaa3474f05/280e86a1-3324-48d8-87d6-419f34121d97"
-					(reference "C?")
+					(reference "C17")
 					(unit 1)
 				)
@@
 		(dnp no)
 		(fields_autoplaced yes)
-		(property "Reference" "C?"
+		(property "Reference" "C16"
 			(at 66.04 53.3399 0)
 			(effects
@@
 			(project "flight_computer"
 				(path "/b71a7b79-cdb5-4e38-a72c-0daaa3474f05/280e86a1-3324-48d8-87d6-419f34121d97"
-					(reference "C?")
+					(reference "C16")
 					(unit 1)
 				)
@@
 		(dnp no)
 		(fields_autoplaced yes)
-		(property "Reference" "C?"
+		(property "Reference" "C18"
 			(at 66.04 104.1399 0)
 			(effects
@@
 			(project "flight_computer"
 				(path "/b71a7b79-cdb5-4e38-a72c-0daaa3474f05/280e86a1-3324-48d8-87d6-419f34121d97"
-					(reference "C?")
+					(reference "C18")
 					(unit 1)
 				)
@@
 		(dnp no)
 		(fields_autoplaced yes)
-		(property "Reference" "C?"
+		(property "Reference" "C19"
 			(at 66.04 129.5399 0)
 			(effects
@@
 			(project "flight_computer"
 				(path "/b71a7b79-cdb5-4e38-a72c-0daaa3474f05/280e86a1-3324-48d8-87d6-419f34121d97"
-					(reference "C?")
-					(unit 1)
-				)
+					(reference "C19")
+					(unit 1)
+				)

Commit message: assigned footprints to capacitors
Parts:
- C12, C13, C14, C15, C16, C17, C18, C19: footprint (none) -> Capacitor_SMD:C_0603_1608Metric
Changed lines of the file:
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@@
 			)
 		)
-		(property "Footprint" ""
+		(property "Footprint" "Capacitor_SMD:C_0603_1608Metric"
 			(at 144.4752 57.15 0)
 			(effects
@@
 			)
 		)
-		(property "Footprint" ""
+		(property "Footprint" "Capacitor_SMD:C_0603_1608Metric"
 			(at 63.1952 83.82 0)
 			(effects
@@
 			)
 		)
-		(property "Footprint" ""
+		(property "Footprint" "Capacitor_SMD:C_0603_1608Metric"
 			(at 158.4452 57.15 0)
 			(effects
@@
 			)
 		)
-		(property "Footprint" ""
+		(property "Footprint" "Capacitor_SMD:C_0603_1608Metric"
 			(at 63.1952 58.42 0)
 			(effects
@@
 			)
 		)
-		(property "Footprint" ""
+		(property "Footprint" "Capacitor_SMD:C_0603_1608Metric"
 			(at 195.2752 86.36 0)
 			(effects
@@
 			)
 		)
-		(property "Footprint" ""
+		(property "Footprint" "Capacitor_SMD:C_0603_1608Metric"
 			(at 183.8452 86.36 0)
 			(effects
@@
 			)
 		)
-		(property "Footprint" ""
+		(property "Footprint" "Capacitor_SMD:C_0603_1608Metric"
 			(at 63.1952 109.22 0)
 			(effects
@@
 			)
 		)
-		(property "Footprint" ""
+		(property "Footprint" "Capacitor_SMD:C_0603_1608Metric"
 			(at 63.1952 134.62 0)
 			(effects

Commit message: net updates
Connections:
- net RTD1A renamed OX_RTD_UPPER_A
- net RTD1B renamed OX_RTD_UPPER_B
- net RTD1C renamed OX_RTD_UPPER_C
- net RTD2A renamed OX_RTD_LOWER_A
- net RTD2B renamed OX_RTD_LOWER_B
- net RTD2C renamed OX_RTD_LOWER_C
Other:
- moved on the sheet: C16, C17, C18, C19
