File: power_systems/voltage_sensing.kicad_sch (KiCad schematic)
At the start: 9 parts, among them U11 OPA333xxD, U12 OPA333xxD, U13 OPA333xxD

Commit message: Power systems routing v1
Parts:
- removed U11, U12, U13: OPA333xxD, Package_SO:SOIC-8_3.9x4.9mm_P1.27mm, symbol Amplifier_Operational:OPA333xxD
Connections:
- net GSE_SENSE: now also R12.2, R13.1
- net VBUCK_SENSE: now also R10.2, R11.1
- net VOUT_SENSE: now also R14.2, R15.1
