File: pyro/pyro_circuit.kicad_sch (KiCad schematic)
At the start: 12 parts, among them Q1 ISA170230C04LMDS, U1 IRLML6344TRPBF

Commit message: bruh
Parts:
- R1: DIGIKEY PART N 541-100HCT-ND -> 311-10.0KHRCT-ND
- R2, R6, R8: DIGIKEY PART N (none) -> RMCF0603FT1K00CT-ND
- R4: DIGIKEY PART N YAG1237CT-ND -> RMCF0603FT1K00CT-ND
- R5: DIGIKEY PART N (none) -> 311-10.0KHRCT-ND
- R7: DIGIKEY PART N (none) -> 2019-RK73B1JTTD202JCT-ND
Changed lines of the file:
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@@
 			)
 		)
-		(property "DIGIKEY PART N" "541-100HCT-ND"
+		(property "DIGIKEY PART N" "311-10.0KHRCT-ND"
 			(at 55.88 86.36 90)
 			(effects
@@
 			)
 		)
-		(property "DIGIKEY PART N" ""
+		(property "DIGIKEY PART N" "RMCF0603FT1K00CT-ND"
 			(at 189.23 100.33 0)
 			(effects
@@
 			)
 		)
-		(property "DIGIKEY PART N" ""
+		(property "DIGIKEY PART N" "RMCF0603FT1K00CT-ND"
 			(at 254 86.36 0)
 			(effects
@@
 			)
 		)
-		(property "DIGIKEY PART N" "YAG1237CT-ND"
+		(property "DIGIKEY PART N" "RMCF0603FT1K00CT-ND"
 			(at 114.3 97.79 0)
 			(effects
@@
 			)
 		)
-		(property "DIGIKEY PART N" ""
+		(property "DIGIKEY PART N" "311-10.0KHRCT-ND"
 			(at 181.61 91.44 90)
 			(effects
@@
 			)
 		)
-		(property "DIGIKEY PART N" ""
+		(property "DIGIKEY PART N" "2019-RK73B1JTTD202JCT-ND "
 			(at 241.3 86.36 0)
 			(effects
@@
 			)
 		)
-		(property "DIGIKEY PART N" ""
+		(property "DIGIKEY PART N" "RMCF0603FT1K00CT-ND"
 			(at 73.66 104.14 90)
 			(effects
